Commit message: Update rover model and Gazebo launch setup

File: src/mars_rover/urdf/rover.urdf.xacro (robot description, xacro)
@@ -3,115 +3,408 @@
     name="mars_rover"
     xmlns:xacro="http://www.ros.org/wiki/xacro">
-    <!-- ====================================================== -->
-    <!-- Include Files                                           -->
-    <!-- ====================================================== -->
-    <xacro:include filename="$(find mars_rover)/urdf/properties.xacro"/>
-    <xacro:include filename="$(find mars_rover)/urdf/materials.xacro"/>
-    <xacro:include filename="$(find mars_rover)/urdf/inertials.xacro"/>
-    <xacro:include filename="$(find mars_rover)/urdf/wheels.xacro"/>
-    <xacro:include filename="$(find mars_rover)/urdf/gazebo.xacro"/>
-    <xacro:include filename="$(find mars_rover)/urdf/ros2_control.xacro"/>
-    <!-- ====================================================== -->
-    <!-- Base Link                                               -->
-    <!-- ====================================================== -->
-<link name="base_link">
+  <!-- ========================================================= -->
+  <!-- Properties / materials / inertials / Gazebo / control      -->
+  <!-- ========================================================= -->
+  <xacro:include filename="$(find mars_rover)/urdf/properties.xacro"/>
+  <xacro:include filename="$(find mars_rover)/urdf/materials.xacro"/>
+  <xacro:include filename="$(find mars_rover)/urdf/inertials.xacro"/>
+  <xacro:include filename="$(find mars_rover)/urdf/gazebo.xacro"/>
+  <xacro:include filename="$(find mars_rover)/urdf/ros2_control.xacro"/>
+  <!-- ========================================================= -->
+  <!-- BASE LINK                                                   -->
+  <!-- ========================================================= -->
+  <link name="base_link">
+    <!-- Main body -->
+   <visual>
+  <origin xyz="0 0 0"
+          rpy="0 0 1.57079632679"/>
+  <geometry>
+    <mesh filename="package://mars_rover/meshes/visual/Main_Body.obj"/>
+  </geometry>
+</visual>
+<visual>
+  <origin xyz="0 0 0"
+          rpy="0 0 1.57079632679"/>
+  <geometry>
+    <mesh filename="package://mars_rover/meshes/visual/Chassis.obj"/>
+  </geometry>
+</visual>
+    <!-- Main collision -->
+    <collision>
+      <origin xyz="0 0 0" rpy="0 0 1.57079632679"/>
+      <geometry>
+        <mesh filename="package://mars_rover/meshes/collision/Main_Body.stl"/>
+      </geometry>
+    </collision>
+    <xacro:box_inertia
+        mass="${body_mass}"
+        x="${body_length}"
+        y="${body_width}"
+        z="${body_height}"/>
+  </link>
+  <!-- ========================================================= -->
+  <!-- CAMERA                                                     -->
+  <!-- ========================================================= -->
+  <link name="camera_link">
+    <visual>
+      <origin xyz="0 0 0" rpy="0 0 1.57079632679"/>
+      <geometry>
+        <mesh filename="package://mars_rover/meshes/visual/ZED2i_Camera.obj"/>
+      </geometry>
+    </visual>
+  </link>
+  <joint name="camera_joint"
+         type="fixed">
+    <parent link="base_link"/>
+    <child link="camera_link"/>
+    <origin xyz="0 0 0"
+            rpy="0 0 0"/>
+  </joint>
+  <link name="camera_optical_frame"/>
+  <joint name="camera_optical_joint"
+         type="fixed">
+    <parent link="camera_link"/>
+    <child link="camera_optical_frame"/>
+    <origin xyz="0 0 0"
+            rpy="-1.570796 0 -1.570796"/>
+  </joint>
+  <!-- ========================================================= -->
+  <!-- FRONT LEFT WHEEL                                            -->
+  <!-- ========================================================= -->
+<!-- ========================================================= -->
+<!-- FRONT LEFT MOTOR                                          -->
+<!-- ========================================================= -->
+<link name="FL_motor_link">
   <visual>
-    <origin xyz="0 0 0" rpy="0 0 0"/>
+    <origin xyz="0 0 0"
+            rpy="0 0 1.57079632679"/>
     <geometry>
-      <mesh filename="package://mars_rover/meshes/visual/Main_Body.obj"/>
+      <mesh filename="package://mars_rover/meshes/visual/Motor_FL.obj"/>
     </geometry>
+    <material name="Silver"/>
   </visual>
-  <visual>
-    <origin xyz="0 0 0" rpy="0 0 0"/>
-    <geometry>
-      <mesh filename="package://mars_rover/meshes/visual/Chassis.obj"/>
-    </geometry>
-  </visual>
-  <collision>
-    <origin xyz="0 0 0" rpy="0 0 0"/>
-    <geometry>
-      <mesh filename="package://mars_rover/meshes/collision/Main_Body.stl"/>
-    </geometry>
-  </collision>
-  <xacro:box_inertia
-    mass="${body_mass}"
-    x="${body_length}"
-    y="${body_width}"
-    z="${body_height}"/>
 </link>
-<link name="camera_link">
-    <visual>
-        <geometry>
-            <mesh filename="package://mars_rover/meshes/visual/ZED2i_Camera.obj"/>
-        </geometry>
-    </visual>
+<joint name="FL_motor_joint"
+       type="fixed">
+  <parent link="base_link"/>
+  <child link="FL_motor_link"/>
+  <origin xyz="0.092373 0.11249 0.063755"
+          rpy="0 0 0"/>
+</joint>
+<!-- ========================================================= -->
+<!-- FRONT LEFT WHEEL                                          -->
+<!-- ========================================================= -->
+<link name="FL_wheel_link">
+<visual>
+  <origin xyz="0 0 0"
+          rpy="0 0 0"/>
+  <geometry>
+    <mesh filename="package://mars_rover/meshes/visual/FL_Wheel.obj"/>
+  </geometry>
+  <material name="Black"/>
+</visual>
+<collision>
+  <origin xyz="0 0 0"
+          rpy="0 0 1.57079632679"/>
+  <geometry>
+    <cylinder
+        radius="${wheel_radius}"
+        length="${wheel_width}"/>
+  </geometry>
+</collision>
+  <xacro:cylinder_inertia
+      mass="${wheel_mass}"
+      radius="${wheel_radius}"
+      length="${wheel_width}"/>
 </link>
-<joint
-name="camera_joint"
-type="fixed">
-<parent link="base_link"/>
-<child link="camera_link"/>
-<origin xyz="0 0 0"/>
+<!-- ========================================================= -->
+<!-- FRONT LEFT WHEEL JOINT                                    -->
+<!-- ========================================================= -->
+<joint name="FL_wheel_joint"
+       type="continuous">
+  <parent link="FL_motor_link"/>
+  <child link="FL_wheel_link"/>
+  <origin xyz="0 0 0"
+          rpy="0 0 1.57079632679"/>
+  <axis xyz="1 0 0"/>
+  <limit effort="30"
+         velocity="30"/>
+  <dynamics damping="0.1"
+            friction="0.1"/>
 </joint>
-<link name="camera_optical_frame"/>
-<joint
-name="camera_optical_joint"
-type="fixed">
-<parent link="camera_link"/>
-<child link="camera_optical_frame"/>
-<origin
-xyz="0 0 0"
-rpy="-1.570796 0 -1.570796"/>
-</joint>
-<!-- ======================================================== -->
-<!-- Wheels -->
-<!-- ======================================================== -->
-<xacro:wheel
-wheel_name="FL"
-parent="base_link"
-wheel_mesh="FL_Wheel"
-motor_mesh="Motor_FL"
-x="${FL_x}"
-y="${FL_y}"
-z="${FL_z}"/>
-<xacro:wheel
-wheel_name="FR"
-parent="base_link"
-wheel_mesh="FR_Wheel"
-motor_mesh="Motor_FR"
-x="${FR_x}"
-y="${FR_y}"
-z="${FR_z}"/>
-<xacro:wheel
-wheel_name="ML"
-parent="base_link"
-wheel_mesh="ML_Wheel"
-motor_mesh="Motor_ML"
-x="${ML_x}"
-y="${ML_y}"
-z="${ML_z}"/>
-<xacro:wheel
-wheel_name="MR"
-parent="base_link"
-wheel_mesh="MR_Wheel"
-motor_mesh="Motor_MR"
-x="${MR_x}"
-y="${MR_y}"
-z="${MR_z}"/>
-<xacro:wheel
-wheel_name="RL"
-parent="base_link"
-wheel_mesh="RL_Wheel"
-motor_mesh="Motor_RL"
-x="${RL_x}"
-y="${RL_y}"
-z="${RL_z}"/>
-<xacro:wheel
-wheel_name="RR"
-parent="base_link"
-wheel_mesh="RR_Wheel"
-motor_mesh="Motor_RR"
-x="${RR_x}"
-y="${RR_y}"
-z="${RR_z}"/>
+  <!-- ========================================================= -->
+  <!-- FRONT RIGHT MOTOR / SUPPORT                                 -->
+  <!-- ========================================================= -->
+  <link name="FR_motor_link">
+    <visual>
+      <origin xyz="0 0 0"
+              rpy="0 1.57079632679 0"/>
+      <geometry>
+        <mesh filename="package://mars_rover/meshes/visual/Motor_FR.obj"/>
+      </geometry>
+    </visual>
+  </link>
+  <joint name="FR_motor_joint"
+         type="fixed">
+    <parent link="base_link"/>
+    <child link="FR_motor_link"/>
+    <origin xyz="0.092373 -0.11309 0.063755"
+            rpy="0 0 0"/>
+  </joint>
+  <link name="FR_wheel_link">
+    <visual>
+      <origin xyz="0 0 0"
+              rpy="0 0 0"/>
+      <geometry>
+        <mesh filename="package://mars_rover/meshes/visual/FR_Wheel.obj"/>
+      </geometry>
+    </visual>
+    <collision>
+      <origin xyz="0 0 0"
+              rpy="0 1.57079632679 0"/>
+      <geometry>
+        <cylinder
+            radius="${wheel_radius}"
+            length="${wheel_width}"/>
+      </geometry>
+    </collision>
+    <xacro:cylinder_inertia
+        mass="${wheel_mass}"
+        radius="${wheel_radius}"
+        length="${wheel_width}"/>
+  </link>
+  <joint name="FR_wheel_joint"
+         type="continuous">
+    <parent link="FR_motor_link"/>
+    <child link="FR_wheel_link"/>
+    <origin xyz="0 0 0"
+            rpy="0 0 1.57079632679"/>
+    <axis xyz="1 0 0"/>
+    <limit
+        effort="30"
+        velocity="30"/>
+    <dynamics
+        damping="0.1"
+        friction="0.1"/>
+  </joint>
+  <!-- ========================================================= -->
+  <!-- MIDDLE LEFT MOTOR / SUPPORT                                -->
+  <!-- ========================================================= -->
+  <link name="ML_motor_link">
+    <visual>
+      <origin xyz="0 0 0"
+              rpy="0 0 1.57079632679"/>
+      <geometry>
+        <mesh filename="package://mars_rover/meshes/visual/Motor_ML.obj"/>
+      </geometry>
+    </visual>
+  </link>
+  <joint name="ML_motor_joint"
+         type="fixed">
+    <parent link="base_link"/>
+    <child link="ML_motor_link"/>
+    <origin xyz="-0.048627 0.11249 0.063755"
+            rpy="0 0 0"/>
+  </joint>
+  <link name="ML_wheel_link">
+    <visual>
+      <origin xyz="0 0 0"
+              rpy="0 0 0"/>
+      <geometry>
+        <mesh filename="package://mars_rover/meshes/visual/ML_Wheel.obj"/>
+      </geometry>
+    </visual>
+    <collision>
+      <origin xyz="0 0 0"
+              rpy="0 1.57079632679 0"/>
+      <geometry>
+        <cylinder
+            radius="${wheel_radius}"
+            length="${wheel_width}"/>
+      </geometry>
+    </collision>
+    <xacro:cylinder_inertia
+        mass="${wheel_mass}"
+        radius="${wheel_radius}"
+        length="${wheel_width}"/>
+  </link>
+  <joint name="ML_wheel_joint"
+         type="continuous">
+    <parent link="ML_motor_link"/>
+    <child link="ML_wheel_link"/>
+    <origin xyz="0 0 0"
+            rpy="0 0 1.57079632679"/>
+    <axis xyz="1 0 0"/>
+    <limit
+        effort="30"
+        velocity="30"/>
+    <dynamics
+        damping="0.1"
+        friction="0.1"/>
+  </joint>
+  <!-- ========================================================= -->
+  <!-- MIDDLE RIGHT MOTOR / SUPPORT                               -->
+  <!-- ========================================================= -->
+  <link name="MR_motor_link">
+    <visual>
+      <origin xyz="0 0 0"
+              rpy="0 0 1.57079632679"/>
+      <geometry>
+        <mesh filename="package://mars_rover/meshes/visual/Motor_MR.obj"/>
+      </geometry>
+    </visual>
+  </link>
+  <joint name="MR_motor_joint"
+         type="fixed">
+    <parent link="base_link"/>
+    <child link="MR_motor_link"/>
+    <origin xyz="-0.048627 -0.11309 0.063755"
+            rpy="0 0 0"/>
+  </joint>
+  <link name="MR_wheel_link">
+    <visual>
+      <origin xyz="0 0 0"
+              rpy="0 0 0"/>
+      <geometry>
+        <mesh filename="package://mars_rover/meshes/visual/MR_Wheel.obj"/>
+      </geometry>
+    </visual>
+    <collision>
+      <origin xyz="0 0 0"
+              rpy="0 1.57079632679 0"/>
+      <geometry>
+        <cylinder
+            radius="${wheel_radius}"
+            length="${wheel_width}"/>
+      </geometry>
+    </collision>
+    <xacro:cylinder_inertia
+        mass="${wheel_mass}"
+        radius="${wheel_radius}"
+        length="${wheel_width}"/>
+  </link>
+  <joint name="MR_wheel_joint"
+         type="continuous">
+    <parent link="MR_motor_link"/>
+    <child link="MR_wheel_link"/>
+    <origin xyz="0 0 0"
+            rpy="0 0 1.57079632679"/>
+    <axis xyz="1 0 0"/>
+    <limit
+        effort="30"
+        velocity="30"/>
+    <dynamics
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
File: src/mars_rover/urdf/wheels.xacro (robot description, xacro)
@@ -1,59 +1,77 @@
 <?xml version="1.0"?>
 <robot xmlns:xacro="http://www.ros.org/wiki/xacro">
-<xacro:macro name="wheel" params="
-    wheel_name
-    parent
-    wheel_mesh
-    motor_mesh
-    x
-    y
-    z">
-  <!-- ================= Motor ================= -->
-  <link name="${wheel_name}_motor_link">
-    <visual>
-      <geometry>
-        <mesh filename="package://mars_rover/meshes/visual/${motor_mesh}.obj"/>
-      </geometry>
-      <material name="Silver"/>
-    </visual>
-  </link>
-  <joint
-      name="${wheel_name}_motor_joint"
-      type="fixed">
+  <xacro:macro name="wheel"
+               params="wheel_name parent wheel_mesh motor_mesh x y z">
+    <!-- ===================================================== -->
+    <!-- FIXED MOTOR LINK                                      -->
+    <!-- ===================================================== -->
+    <link name="${wheel_name}_motor_link">
+      <visual>
+        <origin xyz="0 0 0"
+                rpy="0 0 0"/>
+        <geometry>
+          <mesh filename="package://mars_rover/meshes/visual/${motor_mesh}.obj"/>
+        </geometry>
+        <material name="Silver"/>
+      </visual>
+    </link>
+    <!-- Motor remains fixed to base_link.
+         Its mesh already contains its physical position. -->
+    <joint name="${wheel_name}_motor_joint"
+           type="fixed">
       <parent link="${parent}"/>
       <child link="${wheel_name}_motor_link"/>
+      <origin xyz="0 0 0"
+              rpy="0 0 0"/>
+    </joint>
+    <!-- ===================================================== -->
+    <!-- WHEEL LINK                                            -->
+    <!-- ===================================================== -->
+    <link name="${wheel_name}_wheel_link">
+      <visual>
+        <!--
+          IMPORTANT:
+          The OBJ already contains its world/rover position.
+          The wheel link frame will now be placed at the axle
+          by the wheel joint below.
+          Therefore subtract the axle position here so the
+          visual stays exactly where it is.
+        -->
+        <origin xyz="${-x} ${-y} ${-z}"
+                rpy="0 0 0"/>
+        <geometry>
+          <mesh filename="package://mars_rover/meshes/visual/${wheel_mesh}.obj"/>
+        </geometry>
+        <material name="Black"/>
+      </visual>
+      <!-- Collision is local to the wheel axle -->
+      <collision>
+        <origin xyz="0 0 0"
+                rpy="0 0 0"/>
+        <geometry>
+          <cylinder
+              radius="${wheel_radius}"
+              length="${wheel_width}"/>
+        </geometry>
+      </collision>
+      <xacro:cylinder_inertia
+          mass="${wheel_mass}"
+          radius="${wheel_radius}"
+          length="${wheel_width}"/>
+    </link>
+    <!-- ===================================================== -->
+    <!-- ACTUAL WHEEL ROTATION JOINT                           -->
+    <!-- ===================================================== -->
+    <joint name="${wheel_name}_wheel_joint"
+           type="continuous">
+      <parent link="${wheel_name}_motor_link"/>
+      <child link="${wheel_name}_wheel_link"/>
+      <!--
+        THIS is the important change.
+        Put the wheel-link frame directly at the physical axle.
+      -->
       <origin xyz="${x} ${y} ${z}"
               rpy="0 0 0"/>
-  </joint>
-  <!-- ================= Wheel ================= -->
-  <link name="${wheel_name}_wheel_link">
-<visual>
-  <origin xyz="0 0 0"
-          rpy="0 0 0"/>
-  <geometry>
-    <mesh filename="package://mars_rover/meshes/visual/${wheel_mesh}.obj"/>
-  </geometry>
-  <material name="Black"/>
-</visual>
-    <collision>
-      <origin rpy="0 1.57079632679 0"/>
-      <geometry>
-        <cylinder
-            radius="${wheel_radius}"
-            length="${wheel_width}"/>
-      </geometry>
-    </collision>
-    <xacro:cylinder_inertia
-        mass="${wheel_mass}"
-        radius="${wheel_radius}"
-        length="${wheel_width}"/>
-  </link>
-  <joint
-      name="${wheel_name}_wheel_joint"
-      type="continuous">
-      <parent link="${wheel_name}_motor_link"/>
-      <child link="${wheel_name}_wheel_link"/>
-      <origin xyz="0 0 0"
-              rpy="0 0 0"/>
+      <!-- Your wheel's native axle is X -->
       <axis xyz="1 0 0"/>
       <limit
@@ -63,5 +81,5 @@
           damping="0.1"
           friction="0.1"/>
-  </joint>
-</xacro:macro>
+    </joint>
+  </xacro:macro>
 </robot>
