Commit message: Finalize Mars rover simulation framework

File: src/mars_rover/urdf/properties.xacro (robot description, xacro)
@@ -1,31 +1,32 @@
 <?xml version="1.0"?>
 <robot xmlns:xacro="http://www.ros.org/wiki/xacro">
-  <!-- ================= BODY ================= -->
-  <xacro:property name="body_length" value="0.35"/>
-  <xacro:property name="body_width"  value="0.25"/>
-  <xacro:property name="body_height" value="0.18"/>
-  <xacro:property name="body_mass" value="7.5"/>
-  <!-- ================= WHEELS ================= -->
-  <xacro:property name="wheel_radius" value="0.0565"/>
-  <xacro:property name="wheel_width" value="0.056"/>
+  <!-- BODY -->
+  <xacro:property name="rover_scale" value="2.20"/>
+<xacro:property name="body_length" value="${0.35 * rover_scale}"/>
+<xacro:property name="body_width"  value="${0.25 * rover_scale}"/>
+<xacro:property name="body_height" value="${0.18 * rover_scale}"/>
+  <xacro:property name="body_mass" value="5.5"/>
+  <!-- WHEELS -->
+<xacro:property name="wheel_radius" value="${0.0565 * rover_scale}"/>
+<xacro:property name="wheel_width" value="${0.056 * rover_scale}"/>
   <xacro:property name="wheel_mass" value="0.35"/>
   <!-- Wheel Coordinates -->
-  <xacro:property name="FL_x" value="0.092373"/>
-  <xacro:property name="FL_y" value="0.11249"/>
-  <xacro:property name="FL_z" value="0.063755"/>
-  <xacro:property name="FR_x" value="0.092373"/>
-  <xacro:property name="FR_y" value="-0.11309"/>
-  <xacro:property name="FR_z" value="0.063755"/>
-  <xacro:property name="ML_x" value="-0.048627"/>
-  <xacro:property name="ML_y" value="0.11249"/>
-  <xacro:property name="ML_z" value="0.063755"/>
-  <xacro:property name="MR_x" value="-0.048627"/>
-  <xacro:property name="MR_y" value="-0.11309"/>
-  <xacro:property name="MR_z" value="0.063755"/>
-  <xacro:property name="RL_x" value="-0.18863"/>
-  <xacro:property name="RL_y" value="0.11249"/>
-  <xacro:property name="RL_z" value="0.063755"/>
-  <xacro:property name="RR_x" value="-0.18863"/>
-  <xacro:property name="RR_y" value="-0.11309"/>
-  <xacro:property name="RR_z" value="0.063755"/>
+<xacro:property name="FL_x" value="${0.092373 * rover_scale}"/>
+<xacro:property name="FL_y" value="${0.11249 * rover_scale}"/>
+<xacro:property name="FL_z" value="${0.063755 * rover_scale}"/>
+<xacro:property name="FR_x" value="${0.092373 * rover_scale}"/>
+<xacro:property name="FR_y" value="${-0.11309 * rover_scale}"/>
+<xacro:property name="FR_z" value="${0.063755 * rover_scale}"/>
+<xacro:property name="ML_x" value="${-0.048627 * rover_scale}"/>
+<xacro:property name="ML_y" value="${0.11249 * rover_scale}"/>
+<xacro:property name="ML_z" value="${0.063755 * rover_scale}"/>
+<xacro:property name="MR_x" value="${-0.048627 * rover_scale}"/>
+<xacro:property name="MR_y" value="${-0.11309 * rover_scale}"/>
+<xacro:property name="MR_z" value="${0.063755 * rover_scale}"/>
+<xacro:property name="RL_x" value="${-0.18863 * rover_scale}"/>
+<xacro:property name="RL_y" value="${0.11249 * rover_scale}"/>
+<xacro:property name="RL_z" value="${0.063755 * rover_scale}"/>
+<xacro:property name="RR_x" value="${-0.18863 * rover_scale}"/>
+<xacro:property name="RR_y" value="${-0.11309 * rover_scale}"/>
+<xacro:property name="RR_z" value="${0.063755 * rover_scale}"/>
 </robot>

File: src/mars_rover/urdf/rover.urdf.xacro (robot description, xacro)
@@ -3,7 +3,5 @@
     name="mars_rover"
     xmlns:xacro="http://www.ros.org/wiki/xacro">
-  <!-- ========================================================= -->
-  <!-- Properties / materials / inertials / Gazebo / control      -->
-  <!-- ========================================================= -->
+  <!-- Properties / materials / inertials / Gazebo / control  -->
   <xacro:include filename="$(find mars_rover)/urdf/properties.xacro"/>
   <xacro:include filename="$(find mars_rover)/urdf/materials.xacro"/>
@@ -11,7 +9,5 @@
   <xacro:include filename="$(find mars_rover)/urdf/gazebo.xacro"/>
   <xacro:include filename="$(find mars_rover)/urdf/ros2_control.xacro"/>
-  <!-- ========================================================= -->
-  <!-- BASE LINK                                                   -->
-  <!-- ========================================================= -->
+  <!-- BASE LINK  -->
   <link name="base_link">
     <!-- Main body -->
@@ -20,6 +16,11 @@
           rpy="0 0 1.57079632679"/>
   <geometry>
-    <mesh filename="package://mars_rover/meshes/visual/Main_Body.obj"/>
+           <mesh
+    filename="package://mars_rover/meshes/visual/Main_Body.obj"
+    scale="${rover_scale} ${rover_scale} ${rover_scale}"/>
   </geometry>
+  <material name="BodyGrey">
+  <color rgba="0.35 0.35 0.35 1.0"/>
+</material>
 </visual>
 <visual>
@@ -27,5 +28,7 @@
           rpy="0 0 1.57079632679"/>
   <geometry>
-    <mesh filename="package://mars_rover/meshes/visual/Chassis.obj"/>
+    <mesh
+    filename="package://mars_rover/meshes/visual/Chassis.obj"
+    scale="${rover_scale} ${rover_scale} ${rover_scale}"/>
   </geometry>
 </visual>
@@ -34,5 +37,7 @@
       <origin xyz="0 0 0" rpy="0 0 1.57079632679"/>
       <geometry>
-        <mesh filename="package://mars_rover/meshes/collision/Main_Body.stl"/>
+      <mesh
+    filename="package://mars_rover/meshes/collision/Main_Body.stl"
+    scale="${rover_scale} ${rover_scale} ${rover_scale}"/>
       </geometry>
     </collision>
@@ -43,12 +48,11 @@
         z="${body_height}"/>
   </link>
-  <!-- ========================================================= -->
-  <!-- CAMERA                                                     -->
-  <!-- ========================================================= -->
+  <!-- CAMERA  -->
   <link name="camera_link">
     <visual>
       <origin xyz="0 0 0" rpy="0 0 1.57079632679"/>
       <geometry>
-        <mesh filename="package://mars_rover/meshes/visual/ZED2i_Camera.obj"/>
+        <mesh filename="package://mars_rover/meshes/visual/ZED2i_Camera.obj"
+        scale="${rover_scale} ${rover_scale} ${rover_scale}"/>
       </geometry>
     </visual>
@@ -58,6 +62,8 @@
     <parent link="base_link"/>
     <child link="camera_link"/>
-    <origin xyz="0 0 0"
-            rpy="0 0 0"/>
+    <origin xyz="${0 * rover_scale}
+         ${0 * rover_scale}
+         ${0 * rover_scale}"
+    rpy="0 0 0"/>
   </joint>
   <link name="camera_optical_frame"/>
@@ -69,10 +75,29 @@
             rpy="-1.570796 0 -1.570796"/>
   </joint>
-  <!-- ========================================================= -->
-  <!-- FRONT LEFT WHEEL                                            -->
-  <!-- ========================================================= -->
-<!-- ========================================================= -->
+<!-- ZED 2i LEFT OPTICAL CENTER   -->
+<link name="zed_left_camera_link"/>
+<joint name="zed_left_camera_joint"
+       type="fixed">
+  <parent link="base_link"/>
+  <child link="zed_left_camera_link"/>
+<origin
+    xyz="${0.15518 * rover_scale}
+         ${-0.058794 * rover_scale}
+         ${0.18 * rover_scale}"
+    rpy="0 0 0"/>
+</joint>
+<!-- ZED 2i RIGHT OPTICAL CENTER  -->
+<link name="zed_right_camera_link"/>
+<joint name="zed_right_camera_joint"
+       type="fixed">
+  <parent link="base_link"/>
+  <child link="zed_right_camera_link"/>
+<origin
+    xyz="${0.15518 * rover_scale}
+         ${0.061206 * rover_scale}
+         ${0.17269 * rover_scale}"
+    rpy="0 0 0"/>
+</joint>
 <!-- FRONT LEFT MOTOR                                          -->
-<!-- ========================================================= -->
 <link name="FL_motor_link">
   <visual>
@@ -80,7 +105,7 @@
             rpy="0 0 1.57079632679"/>
     <geometry>
-      <mesh filename="package://mars_rover/meshes/visual/Motor_FL.obj"/>
+      <mesh filename="package://mars_rover/meshes/visual/Motor_FL.obj"
+      scale="${rover_scale} ${rover_scale} ${rover_scale}"/>
     </geometry>
-    <material name="Silver"/>
   </visual>
 </link>
@@ -89,10 +114,10 @@
   <parent link="base_link"/>
   <child link="FL_motor_link"/>
-  <origin xyz="0.092373 0.11249 0.063755"
+  <origin xyz="${0.092373 * rover_scale}
+         ${0.11249 * rover_scale}
+         ${0.063755 * rover_scale}"
           rpy="0 0 0"/>
 </joint>
-<!-- ========================================================= -->
-<!-- FRONT LEFT WHEEL                                          -->
-<!-- ========================================================= -->
+<!-- FRONT LEFT WHEEL -->
 <link name="FL_wheel_link">
 <visual>
@@ -100,11 +125,11 @@
           rpy="0 0 0"/>
   <geometry>
-    <mesh filename="package://mars_rover/meshes/visual/FL_Wheel.obj"/>
+    <mesh filename="package://mars_rover/meshes/visual/FL_Wheel.obj"
+    scale="${rover_scale} ${rover_scale} ${rover_scale}"/>
   </geometry>
-  <material name="Black"/>
 </visual>
 <collision>
   <origin xyz="0 0 0"
-          rpy="0 0 1.57079632679"/>
+          rpy="0 1.57079632679 0"/>
   <geometry>
     <cylinder
@@ -118,7 +143,5 @@
       length="${wheel_width}"/>
 </link>
-<!-- ========================================================= -->
-<!-- FRONT LEFT WHEEL JOINT                                    -->
-<!-- ========================================================= -->
+<!-- FRONT LEFT WHEEL JOINT -->
 <joint name="FL_wheel_joint"
        type="continuous">
@@ -133,13 +156,12 @@
             friction="0.1"/>
 </joint>
-  <!-- ========================================================= -->
-  <!-- FRONT RIGHT MOTOR / SUPPORT                                 -->
-  <!-- ========================================================= -->
+  <!-- FRONT RIGHT MOTOR / SUPPORT  -->
   <link name="FR_motor_link">
     <visual>
       <origin xyz="0 0 0"
-              rpy="0 1.57079632679 0"/>
-      <geometry>
-        <mesh filename="package://mars_rover/meshes/visual/Motor_FR.obj"/>
+              rpy="0 0 1.57079632679"/>
+      <geometry>
+        <mesh filename="package://mars_rover/meshes/visual/Motor_FR.obj"
+        scale="${rover_scale} ${rover_scale} ${rover_scale}"/>
       </geometry>
     </visual>
@@ -149,6 +171,8 @@
     <parent link="base_link"/>
     <child link="FR_motor_link"/>
-    <origin xyz="0.092373 -0.11309 0.063755"
-            rpy="0 0 0"/>
+       <origin xyz="${0.092373 * rover_scale}
+         ${-0.11309 * rover_scale}
+         ${0.063755 * rover_scale}"
+          rpy="0 0 0"/>
   </joint>
   <link name="FR_wheel_link">
@@ -157,5 +181,6 @@
               rpy="0 0 0"/>
       <geometry>
-        <mesh filename="package://mars_rover/meshes/visual/FR_Wheel.obj"/>
+        <mesh filename="package://mars_rover/meshes/visual/FR_Wheel.obj"
+        scale="${rover_scale} ${rover_scale} ${rover_scale}"/>
       </geometry>
     </visual>
@@ -188,7 +213,5 @@
         friction="0.1"/>
   </joint>
-  <!-- ========================================================= -->
-  <!-- MIDDLE LEFT MOTOR / SUPPORT                                -->
-  <!-- ========================================================= -->
+  <!-- MIDDLE LEFT MOTOR / SUPPORT -->
   <link name="ML_motor_link">
     <visual>
@@ -196,5 +219,6 @@
               rpy="0 0 1.57079632679"/>
       <geometry>
-        <mesh filename="package://mars_rover/meshes/visual/Motor_ML.obj"/>
+        <mesh filename="package://mars_rover/meshes/visual/Motor_ML.obj"
+        scale="${rover_scale} ${rover_scale} ${rover_scale}"/>
       </geometry>
     </visual>
@@ -204,6 +228,8 @@
     <parent link="base_link"/>
     <child link="ML_motor_link"/>
-    <origin xyz="-0.048627 0.11249 0.063755"
-            rpy="0 0 0"/>
+      <origin xyz="${-0.048627 * rover_scale}
+         ${0.11249 * rover_scale}
+         ${0.063755 * rover_scale}"
+          rpy="0 0 0"/>
   </joint>
   <link name="ML_wheel_link">
@@ -212,5 +238,6 @@
               rpy="0 0 0"/>
       <geometry>
-        <mesh filename="package://mars_rover/meshes/visual/ML_Wheel.obj"/>
+        <mesh filename="package://mars_rover/meshes/visual/ML_Wheel.obj"
+        scale="${rover_scale} ${rover_scale} ${rover_scale}"/>
       </geometry>
     </visual>
@@ -243,7 +270,5 @@
         friction="0.1"/>
   </joint>
-  <!-- ========================================================= -->
-  <!-- MIDDLE RIGHT MOTOR / SUPPORT                               -->
-  <!-- ========================================================= -->
+  <!-- MIDDLE RIGHT MOTOR / SUPPORT  -->
   <link name="MR_motor_link">
     <visual>
@@ -251,5 +276,6 @@
               rpy="0 0 1.57079632679"/>
       <geometry>
-        <mesh filename="package://mars_rover/meshes/visual/Motor_MR.obj"/>
+        <mesh filename="package://mars_rover/meshes/visual/Motor_MR.obj"
+        scale="${rover_scale} ${rover_scale} ${rover_scale}"/>
       </geometry>
     </visual>
@@ -259,6 +285,8 @@
     <parent link="base_link"/>
     <child link="MR_motor_link"/>
-    <origin xyz="-0.048627 -0.11309 0.063755"
-            rpy="0 0 0"/>
+         <origin xyz="${-0.048627 * rover_scale}
+         ${-0.11309 * rover_scale}
+         ${0.063755 * rover_scale}"
+          rpy="0 0 0"/>
   </joint>
   <link name="MR_wheel_link">
@@ -267,5 +295,6 @@
               rpy="0 0 0"/>
       <geometry>
-        <mesh filename="package://mars_rover/meshes/visual/MR_Wheel.obj"/>
+        <mesh filename="package://mars_rover/meshes/visual/MR_Wheel.obj"
+        scale="${rover_scale} ${rover_scale} ${rover_scale}"/>
       </geometry>
     </visual>
@@ -298,7 +327,5 @@
         friction="0.1"/>
   </joint>
-  <!-- ========================================================= -->
-  <!-- REAR LEFT MOTOR / SUPPORT                                  -->
-  <!-- ========================================================= -->
+  <!-- REAR LEFT MOTOR / SUPPORT -->
   <link name="RL_motor_link">
     <visual>
@@ -306,5 +333,6 @@
               rpy="0 0 1.57079632679"/>
       <geometry>
-        <mesh filename="package://mars_rover/meshes/visual/Motor_RL.obj"/>
+        <mesh filename="package://mars_rover/meshes/visual/Motor_RL.obj"
+        scale="${rover_scale} ${rover_scale} ${rover_scale}"/>
       </geometry>
     </visual>
@@ -314,6 +342,8 @@
     <parent link="base_link"/>
     <child link="RL_motor_link"/>
-    <origin xyz="-0.18863 0.11249 0.063755"
-            rpy="0 0 0"/>
+           <origin xyz="${-0.18863 * rover_scale}
+         ${0.11249 * rover_scale}
+         ${0.063755 * rover_scale}"
+          rpy="0 0 0"/>
   </joint>
   <link name="RL_wheel_link">
@@ -322,5 +352,6 @@
               rpy="0 0 0"/>
       <geometry>
-        <mesh filename="package://mars_rover/meshes/visual/RL_Wheel.obj"/>
+        <mesh filename="package://mars_rover/meshes/visual/RL_Wheel.obj"
+        scale="${rover_scale} ${rover_scale} ${rover_scale}"/>
       </geometry>
     </visual>
@@ -353,7 +384,5 @@
         friction="0.1"/>
   </joint>
-  <!-- ========================================================= -->
-  <!-- REAR RIGHT MOTOR / SUPPORT                                 -->
-  <!-- ========================================================= -->
+  <!-- REAR RIGHT MOTOR / SUPPORT -->
   <link name="RR_motor_link">
     <visual>
@@ -361,5 +390,6 @@
               rpy="0 0 1.57079632679"/>
       <geometry>
-        <mesh filename="package://mars_rover/meshes/visual/Motor_RR.obj"/>
+        <mesh filename="package://mars_rover/meshes/visual/Motor_RR.obj"
+        scale="${rover_scale} ${rover_scale} ${rover_scale}"/>
       </geometry>
     </visual>
@@ -369,6 +399,8 @@
     <parent link="base_link"/>
     <child link="RR_motor_link"/>
-    <origin xyz="-0.18863 -0.11309 0.063755"
-            rpy="0 0 0"/>
+        <origin xyz="${-0.18863 * rover_scale}
+         ${-0.11309 * rover_scale}
+         ${0.063755 * rover_scale}"
+          rpy="0 0 0"/>
   </joint>
   <link name="RR_wheel_link">
@@ -377,5 +409,6 @@
               rpy="0 0 0"/>
       <geometry>
-        <mesh filename="package://mars_rover/meshes/visual/RR_Wheel.obj"/>
+        <mesh filename="package://mars_rover/meshes/visual/RR_Wheel.obj"
+        scale="${rover_scale} ${rover_scale} ${rover_scale}"/>
       </geometry>
     </visual>
@@ -408,3 +441,134 @@
         friction="0.1"/>
   </joint>
+<!-- ZED 2i LEFT CAMERA SENSOR  -->
+<gazebo reference="zed_left_camera_link">
+  <sensor
+      name="zed_left_camera"
+      type="camera">
+    <pose>0 0 0 0 0 0</pose>
+    <always_on>true</always_on>
+    <update_rate>15</update_rate>
+    <visualize>false</visualize>
+    <camera>
+      <horizontal_fov>1.7628</horizontal_fov>
+      <image>
+        <width>640</width>
+        <height>360</height>
+        <format>R8G8B8</format>
+      </image>
+      <clip>
+        <near>0.05</near>
+        <far>100.0</far>
+      </clip>
+    </camera>
+    <topic>/zed/zed_node/left/image_rect_color</topic>
+  </sensor>
+</gazebo>
+<!-- ZED 2i RIGHT CAMERA SENSOR  -->
+<gazebo reference="zed_right_camera_link">
+  <sensor
+      name="zed_right_camera"
+      type="camera">
+    <pose>0 0 0 0 0 0</pose>
+    <always_on>true</always_on>
+    <update_rate>15</update_rate>
+    <visualize>false</visualize>
+    <camera>
+      <horizontal_fov>1.7628</horizontal_fov>
+      <image>
+        <width>640</width>
+        <height>360</height>
+        <format>R8G8B8</format>
+      </image>
+      <clip>
+        <near>0.05</near>
+        <far>100.0</far>
+      </clip>
+    </camera>
+    <topic>/zed/zed_node/right/image_rect_color</topic>
+  </sensor>
+</gazebo>
+<gazebo>
+  <plugin
+      filename="gz-sim-diff-drive-system"
+      name="gz::sim::systems::DiffDrive">
+    <left_joint>FL_wheel_joint</left_joint>
+    <left_joint>ML_wheel_joint</left_joint>
+    <left_joint>RL_wheel_joint</left_joint>
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
File: src/mars_rover/urdf/wheels.xacro (robot description, xacro)
@@ -3,7 +3,5 @@
   <xacro:macro name="wheel"
                params="wheel_name parent wheel_mesh motor_mesh x y z">
-    <!-- ===================================================== -->
-    <!-- FIXED MOTOR LINK                                      -->
-    <!-- ===================================================== -->
+    <!-- FIXED MOTOR LINK  -->
     <link name="${wheel_name}_motor_link">
       <visual>
@@ -16,6 +14,4 @@
       </visual>
     </link>
-    <!-- Motor remains fixed to base_link.
-         Its mesh already contains its physical position. -->
     <joint name="${wheel_name}_motor_joint"
            type="fixed">
@@ -25,17 +21,7 @@
               rpy="0 0 0"/>
     </joint>
-    <!-- ===================================================== -->
-    <!-- WHEEL LINK                                            -->
-    <!-- ===================================================== -->
+    <!-- WHEEL LINK   -->
     <link name="${wheel_name}_wheel_link">
       <visual>
-        <!--
-          IMPORTANT:
-          The OBJ already contains its world/rover position.
-          The wheel link frame will now be placed at the axle
-          by the wheel joint below.
-          Therefore subtract the axle position here so the
-          visual stays exactly where it is.
-        -->
         <origin xyz="${-x} ${-y} ${-z}"
                 rpy="0 0 0"/>
@@ -60,18 +46,12 @@
           length="${wheel_width}"/>
     </link>
-    <!-- ===================================================== -->
-    <!-- ACTUAL WHEEL ROTATION JOINT                           -->
-    <!-- ===================================================== -->
+    <!-- WHEEL ROTATION JOINT  -->
     <joint name="${wheel_name}_wheel_joint"
            type="continuous">
       <parent link="${wheel_name}_motor_link"/>
       <child link="${wheel_name}_wheel_link"/>
-      <!--
-        THIS is the important change.
-        Put the wheel-link frame directly at the physical axle.
-      -->
       <origin xyz="${x} ${y} ${z}"
               rpy="0 0 0"/>
-      <!-- Your wheel's native axle is X -->
+      <!-- wheel's native axle is X -->
       <axis xyz="1 0 0"/>
       <limit
